Commit message: Port remaining CUCR worlds, Reachy Zuuu base, and parked TF RELIABLE QoS.
house_museum keeps the CUCR sunset sky with roofs stripped; small_house and small_warehouse sanitize Assimp Material #N names so maps survive convert.

File: src/config/robots/reachy/reachy.urdf (robot description, URDF)
Before this commit: robot reachy_2023, 36 links, 35 joints
Links:
- removed link world
- added link bar_link; collision cylinder length=0.775 radius=0.02; visual cylinder length=0.775 radius=0.02
- added link base_footprint
- added link base_link, mass 24.0; collision cylinder length=0.19 radius=0.245; visual mesh filename=file:///home/osamuzahid/Projects/isaac-social-nav/ros2_ws/s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
- added link drivewhl1_link, mass 0.5; collision cylinder length=0.035 radius=0.105; visual cylinder length=0.035 radius=0.105
- added link drivewhl2_link, mass 0.5; collision cylinder length=0.035 radius=0.105; visual cylinder length=0.035 radius=0.105
- added link drivewhl3_link, mass 0.5; collision cylinder length=0.035 radius=0.105; visual cylinder length=0.035 radius=0.105
- added link imu_link
- added link lidar_link, mass 0.125; collision cylinder length=0.035 radius=0.035
Joints:
- removed joint world_joint
- added joint bar_joint: type fixed, parent base_link, child bar_link, origin xyz=-0.130 0 0.0 rpy=0 0 0
- added joint base_footprint_joint: type fixed, parent base_footprint, child base_link, origin xyz=0 0 0 rpy=0 0 0
- added joint base_joint: type fixed, parent base_link, child torso, origin xyz=-0.006 0 1.0 rpy=0 0 0
- added joint drivewhl1_joint: type fixed, parent base_link, child drivewhl1_link, origin xyz=0.09900000000000003 -0.17147302994931884 0.105 rpy=0 0 0.5235987755982989, axis 0 1 0
- added joint drivewhl2_joint: type fixed, parent base_link, child drivewhl2_link, origin xyz=0.09900000000000003 0.17147302994931884 0.105 rpy=0 0 -3.6651914291880923, axis 0 1 0
- added joint drivewhl3_joint: type fixed, parent base_link, child drivewhl3_link, origin xyz=-0.198 -2.4248006623117595e-17 0.105 rpy=0 0 -1.5707963267948966, axis 0 1 0
- added joint imu_joint: type fixed, parent base_link, child imu_link, origin xyz=0 0 0.01
- added joint lidar_joint: type fixed, parent base_link, child lidar_link, origin xyz=0.184 0 0.25 rpy=0 0 0

File: src/config/robots/reachy/urdf/reachy.urdf.xacro (robot description, xacro)
@@ -8,9 +8,31 @@
   <xacro:include filename="/home/osamuzahid/Projects/isaac-social-nav/ros2_ws/src/Hunav_isaac_wrapper/src/config/robots/reachy/urdf/head.urdf.xacro"/>
   <xacro:include filename="/home/osamuzahid/Projects/isaac-social-nav/ros2_ws/src/Hunav_isaac_wrapper/src/config/robots/reachy/urdf/orbita.urdf.xacro"/>
-  <link name="world"/>
-  <joint name="world_joint" type="fixed">
-    <origin xyz="0 0 1.0" rpy="0 0 0"/>
-    <parent link="world"/>
+  <xacro:include filename="/home/osamuzahid/Projects/isaac-social-nav/ros2_ws/src/Hunav_isaac_wrapper/src/config/robots/reachy/urdf/zuuu.urdf.xacro"/>
+  <!-- PATCH (isaac-social-nav): Zuuu mobile base (lab Reachy). Torso sits on
+       the pole — not world→torso at z=1.0 (Phase 0 table-top). -->
+  <xacro:zuuu/>
+  <joint name="base_joint" type="fixed">
+    <origin xyz="-0.006 0 1.0" rpy="0 0 0"/>
+    <parent link="base_link"/>
     <child link="torso"/>
+  </joint>
+  <link name="bar_link">
+    <visual>
+      <origin xyz="0.0 0.0 0.6125" rpy="0.0 0.0 0.0"/>
+      <geometry>
+        <cylinder radius="0.02" length="0.775"/>
+      </geometry>
+    </visual>
+    <collision>
+      <origin xyz="0.0 0.0 0.6125" rpy="0.0 0.0 0.0"/>
+      <geometry>
+        <cylinder radius="0.02" length="0.775"/>
+      </geometry>
+    </collision>
+  </link>
+  <joint name="bar_joint" type="fixed">
+    <origin xyz="-0.130 0 0.0" rpy="0 0 0"/>
+    <parent link="base_link"/>
+    <child link="bar_link"/>
   </joint>
   <link name="torso">
